Commit message: Fixed URDF to support macros, Updated README, Updated Plot script

File: urdf/gripper.urdf.xacro (robot description, xacro)
@@ -1,35 +1,10 @@
 <?xml version="1.0"?>
-<robot xmlns:xacro="http://www.ros.org/wiki/xacro" name="test">
+<robot xmlns:xacro="http://www.ros.org/wiki/xacro" name="pinc_open">
   <xacro:arg name="use_mock_hardware" default="false" />
-  <xacro:arg name="mock_sensor_commands" default="false" />
-  <xacro:arg name="sim_gazebo" default="false" />
-  <!-- Include links and joints -->
-  <xacro:include filename="gripper_links.xacro"/>
+  <xacro:arg name="prefix" default=""/>
   <xacro:include filename="gripper_macros.xacro"/>
-  <!-- ros2_control -->
-  <ros2_control name="test" type="system">
-    <hardware>
-      <xacro:if value="$(arg use_mock_hardware)">
-        <plugin>mock_components/GenericSystem</plugin>
-      </xacro:if>
-      <xacro:unless value="$(arg use_mock_hardware)">
-        <plugin>pinc_open_driver/PincOpenDriver</plugin>
-        <param name="port">/dev/pinc-gripper</param>
-        <param name="baud_rate">1000000</param>
-        <param name="id">6</param>
-      </xacro:unless>
-    </hardware>
-    <joint name="gripper">
-      <command_interface name="position">
-        <param name="min">-2.44</param>
-        <param name="max">0.0</param>
-      </command_interface>
-      <state_interface name="position">
-        <param name="initial_value">0.0</param>
-      </state_interface>
-      <state_interface name="velocity">
-        <param name="initial_value">0.0</param>
-      </state_interface>
-    </joint>
-  </ros2_control>
+  <xacro:pinc_open_gripper
+    name="pinc_open"
+    use_mock_hardware="$(arg use_mock_hardware)"
+    prefix="$(arg prefix)" />
 </robot>

File: urdf/gripper_links.xacro (robot description, xacro)
@@ -1,8 +1,10 @@
 <?xml version="1.0"?>
 <robot xmlns:xacro="http://www.ros.org/wiki/xacro">
+  <xacro:arg name="prefix" default=""/>
   <!-- Properties -->
   <xacro:property name="mesh_scale" value="0.001 0.001 0.001"/>
+  <xacro:property name="default_color_rgba" value="0 0 1.0 1.0"/>
   <!-- Macros -->
-  <xacro:macro name="visual_mesh" params="mesh_file color_rgba">
+  <xacro:macro name="visual_mesh" params="mesh_file color_rgba:=${default_color_rgba}">
     <visual>
       <geometry>
@@ -14,20 +16,19 @@
     </visual>
   </xacro:macro>
-  <!-- Links -->
-  <link name="base_link">
-    <xacro:visual_mesh mesh_file="package://pinc_open_driver/meshes/Gripper_Palm_Shell_w_motor_v1.stl" color_rgba="0 0 1 1"/>
+  <link name="${prefix}base_link">
+    <xacro:visual_mesh mesh_file="package://pinc_open_driver/meshes/Gripper_Palm_Shell_w_motor_v1.stl"/>
   </link>
-  <link name="coupler"/>
-  <link name="right_arm">
+  <link name="${prefix}coupler"/>
+  <link name="${prefix}right_arm">
     <xacro:visual_mesh mesh_file="package://pinc_open_driver/meshes/gripper_right_arm.stl" color_rgba="0.0 0.5 1.0 1.0"/>
   </link>
-  <link name="left_arm">
+  <link name="${prefix}left_arm">
     <xacro:visual_mesh mesh_file="package://pinc_open_driver/meshes/gripper_left_arm.stl" color_rgba="0.0 0.5 1.0 1.0"/>
   </link>
-  <link name="right_finger">
-    <xacro:visual_mesh mesh_file="package://pinc_open_driver/meshes/gripper_right_finger.stl" color_rgba="0 0 1 1"/>
+  <link name="${prefix}right_finger">
+    <xacro:visual_mesh mesh_file="package://pinc_open_driver/meshes/gripper_right_finger.stl"/>
   </link>
-  <link name="left_finger">
-    <xacro:visual_mesh mesh_file="package://pinc_open_driver/meshes/gripper_left_finger.stl" color_rgba="0 0 1 1"/>
+  <link name="${prefix}left_finger">
+    <xacro:visual_mesh mesh_file="package://pinc_open_driver/meshes/gripper_left_finger.stl"/>
   </link>
 </robot>

File: urdf/gripper_macros.xacro (robot description, xacro)
@@ -1,43 +1,77 @@
 <?xml version="1.0"?>
 <robot xmlns:xacro="http://www.ros.org/wiki/xacro">
-  <!-- Joints -->
-  <joint name="gripper" type="revolute">
-    <parent link="base_link"/>
-    <child link="coupler"/>
+  <xacro:macro name="pinc_open_gripper" params="
+                name
+                prefix
+                use_mock_hardware:=^|false"
+  >
+  <!-- Include links and joints -->
+  <xacro:include filename="$(find pinc_open_driver)/urdf/gripper_links.xacro"/>
+   <!-- Joints -->
+  <joint name="${prefix}gripper" type="revolute">
+    <parent link="${prefix}base_link"/>
+    <child link="${prefix}coupler"/>
     <origin xyz="0.053492 0 0.0"/>
     <axis xyz="0 0 1"/>
     <limit lower="-2.44" upper="0" effort="5" velocity="1"/>
   </joint>
-  <joint name="base_link_to_right_arm" type="revolute">
-    <parent link="base_link"/>
-    <child link="right_arm"/>
+  <joint name="${prefix}base_link_to_right_arm" type="revolute">
+    <parent link="${prefix}base_link"/>
+    <child link="${prefix}right_arm"/>
     <origin xyz="0.053492 -0.03250 -0.008"/>
     <axis xyz="0 0 1"/>
     <limit lower="-1.22" upper="0" effort="5" velocity="1"/>
-    <mimic joint="gripper" multiplier="0.5" offset="0.0"/>
+    <mimic joint="${prefix}gripper" multiplier="0.5" offset="0.0"/>
   </joint>
-  <joint name="base_link_to_left_arm" type="revolute">
-    <parent link="base_link"/>
-    <child link="left_arm"/>
+  <joint name="${prefix}base_link_to_left_arm" type="revolute">
+    <parent link="${prefix}base_link"/>
+    <child link="${prefix}left_arm"/>
     <origin xyz="0.053492 0.03250 -0.008"/>
     <axis xyz="0 0 1"/>
     <limit lower="1.22" upper="0" effort="5" velocity="1"/>
-    <mimic joint="gripper" multiplier="-0.5" offset="0.0"/>
+    <mimic joint="${prefix}gripper" multiplier="-0.5" offset="0.0"/>
   </joint>
-  <joint name="right_arm_to_right_finger" type="revolute">
-    <parent link="right_arm"/>
-    <child link="right_finger"/>
+  <joint name="${prefix}right_arm_to_right_finger" type="revolute">
+    <parent link="${prefix}right_arm"/>
+    <child link="${prefix}right_finger"/>
     <origin xyz="0.034641 0.020 -0.0002"/>
     <axis xyz="0 0 1"/>
     <limit lower="1.22" upper="0" effort="5" velocity="1"/>
-    <mimic joint="gripper" multiplier="-0.5" offset="0.0"/>
+    <mimic joint="${prefix}gripper" multiplier="-0.5" offset="0.0"/>
   </joint>
-  <joint name="left_arm_to_left_finger" type="revolute">
-    <parent link="left_arm"/>
-    <child link="left_finger"/>
+  <joint name="${prefix}left_arm_to_left_finger" type="revolute">
+    <parent link="${prefix}left_arm"/>
+    <child link="${prefix}left_finger"/>
     <origin xyz="0.034641 -0.020 0.0002"/>
     <axis xyz="0 0 1"/>
     <limit lower="-1.22" upper="0" effort="5" velocity="1"/>
-    <mimic joint="gripper" multiplier="0.5" offset="0.0"/>
+    <mimic joint="${prefix}gripper" multiplier="0.5" offset="0.0"/>
   </joint>
+  <!-- ros2_control -->
+  <ros2_control name="${prefix}ros2_control" type="system">
+    <hardware>
+      <xacro:if value="${use_mock_hardware}">
+        <plugin>mock_components/GenericSystem</plugin>
+      </xacro:if>
+      <xacro:unless value="${use_mock_hardware}">
+        <plugin>pinc_open_driver/PincOpenDriver</plugin>
+        <param name="port">/dev/pinc-gripper</param>
+        <param name="baud_rate">1000000</param>
+        <param name="id">6</param>
+      </xacro:unless>
+    </hardware>
+    <joint name="${prefix}gripper">
+      <command_interface name="position">
+        <param name="min">-2.44</param>
+        <param name="max">0.0</param>
+      </command_interface>
+      <state_interface name="position">
+        <param name="initial_value">0.0</param>
+      </state_interface>
+      <state_interface name="velocity">
+        <param name="initial_value">0.0</param>
+      </state_interface>
+    </joint>
+  </ros2_control>
+  </xacro:macro>
 </robot>

Commit message: Use color arguments in URDF to allow change from outside; use joint name to retrieve parameters in cpp

File: urdf/gripper.urdf.xacro (robot description, xacro)
@@ -3,8 +3,15 @@
   <xacro:arg name="use_mock_hardware" default="false" />
   <xacro:arg name="prefix" default=""/>
+  <xacro:arg name="default_color_rgba" default="0 0 1.0 1.0"/>
+  <xacro:arg name="default_linkage_color_rgba" default="0 0.5 1.0 1.0"/>
+  <xacro:arg name="default_tip_color_rgba" default="0 0.0 1.0 1.0"/>
   <xacro:include filename="gripper_macros.xacro"/>
   <xacro:pinc_open_gripper
     name="pinc_open"
     use_mock_hardware="$(arg use_mock_hardware)"
-    prefix="$(arg prefix)" />
+    prefix="$(arg prefix)"
+    default_color_rgba="$(arg default_color_rgba)"
+    default_linkage_color_rgba="$(arg default_linkage_color_rgba)"
+    default_tip_color_rgba="$(arg default_tip_color_rgba)"
+  />
 </robot>

File: urdf/gripper_links.xacro (robot description, xacro)
@@ -2,7 +2,9 @@
 <robot xmlns:xacro="http://www.ros.org/wiki/xacro">
   <xacro:arg name="prefix" default=""/>
+  <xacro:arg name="default_color_rgba" default="0 0 1.0 1.0"/>
+  <xacro:arg name="default_linkage_color_rgba" default="0 0.5 1.0 1.0"/>
+  <xacro:arg name="default_tip_color_rgba" default="0 0.0 1.0 1.0"/>
   <!-- Properties -->
   <xacro:property name="mesh_scale" value="0.001 0.001 0.001"/>
-  <xacro:property name="default_color_rgba" value="0 0 1.0 1.0"/>
   <!-- Macros -->
   <xacro:macro name="visual_mesh" params="mesh_file color_rgba:=${default_color_rgba}">
@@ -21,14 +23,14 @@
   <link name="${prefix}coupler"/>
   <link name="${prefix}right_arm">
-    <xacro:visual_mesh mesh_file="package://pinc_open_driver/meshes/gripper_right_arm.stl" color_rgba="0.0 0.5 1.0 1.0"/>
+    <xacro:visual_mesh mesh_file="package://pinc_open_driver/meshes/gripper_right_arm.stl" color_rgba="${default_linkage_color_rgba}"/>
   </link>
   <link name="${prefix}left_arm">
-    <xacro:visual_mesh mesh_file="package://pinc_open_driver/meshes/gripper_left_arm.stl" color_rgba="0.0 0.5 1.0 1.0"/>
+    <xacro:visual_mesh mesh_file="package://pinc_open_driver/meshes/gripper_left_arm.stl" color_rgba="${default_linkage_color_rgba}"/>
   </link>
   <link name="${prefix}right_finger">
-    <xacro:visual_mesh mesh_file="package://pinc_open_driver/meshes/gripper_right_finger.stl"/>
+    <xacro:visual_mesh mesh_file="package://pinc_open_driver/meshes/gripper_right_finger.stl" color_rgba="${default_tip_color_rgba}"/>
   </link>
   <link name="${prefix}left_finger">
-    <xacro:visual_mesh mesh_file="package://pinc_open_driver/meshes/gripper_left_finger.stl"/>
+    <xacro:visual_mesh mesh_file="package://pinc_open_driver/meshes/gripper_left_finger.stl" color_rgba="${default_tip_color_rgba}"/>
   </link>
 </robot>

File: urdf/gripper_macros.xacro (robot description, xacro)
@@ -4,5 +4,8 @@
                 name
                 prefix
-                use_mock_hardware:=^|false"
+                use_mock_hardware:=^|false
+                default_color_rgba:='0 0 1. 1.'
+                default_linkage_color_rgba:='0 0.5 1.0 1.0'
+                default_tip_color_rgba:='0 0 1. 1.'"
   >
   <!-- Include links and joints -->
@@ -37,5 +40,5 @@
     <origin xyz="0.034641 0.020 -0.0002"/>
     <axis xyz="0 0 1"/>
-    <limit lower="1.22" upper="0" effort="5" velocity="1"/>
+    <limit lower="0" upper="1.22" effort="5" velocity="1"/>
     <mimic joint="${prefix}gripper" multiplier="-0.5" offset="0.0"/>
   </joint>

Commit message: add additional launch arguments; update on_configure/on_shutdown logic; use namespace; flake8, cpplint, and ament_clang_format clean up;

File: urdf/gripper.urdf.xacro (robot description, xacro)
@@ -6,8 +6,19 @@
   <xacro:arg name="default_linkage_color_rgba" default="0 0.5 1.0 1.0"/>
   <xacro:arg name="default_tip_color_rgba" default="0 0.0 1.0 1.0"/>
-  <xacro:arg name="motor_id" default="6"/>
+  <xacro:arg name="baud_rate" default="1000000"/>
+  <xacro:arg name="comm_config_delay_ms" default="100"/>
   <xacro:arg name="serial_port" default="/dev/pinc-gripper"/>
+  <xacro:arg name="serial_timeout" default="50"/>
+  <xacro:arg name="servo_id" default="6"/>
   <xacro:include filename="gripper_macros.xacro"/>
+  <xacro:include filename="gripper_ros2_control.xacro"/>
   <xacro:pinc_open_gripper
+    name="pinc_open"
+    prefix="$(arg prefix)"
+    default_color_rgba="$(arg default_color_rgba)"
+    default_linkage_color_rgba="$(arg default_linkage_color_rgba)"
+    default_tip_color_rgba="$(arg default_tip_color_rgba)"
+  />
+  <xacro:pinc_open_ros2_control
     name="pinc_open"
     use_mock_hardware="$(arg use_mock_hardware)"
@@ -16,6 +27,9 @@
     default_linkage_color_rgba="$(arg default_linkage_color_rgba)"
     default_tip_color_rgba="$(arg default_tip_color_rgba)"
-    motor_id="$(arg motor_id)"
+    baud_rate="$(arg baud_rate)"
+    comm_config_delay_ms="$(arg comm_config_delay_ms)"
     serial_port="$(arg serial_port)"
+    serial_timeout="$(arg serial_timeout)"
+    servo_id="$(arg servo_id)"
   />
 </robot>

File: urdf/gripper_macros.xacro (robot description, xacro)
@@ -4,10 +4,8 @@
                 name
                 prefix
-                use_mock_hardware:=^|false
                 default_color_rgba:='0 0 1. 1.'
                 default_linkage_color_rgba:='0 0.5 1.0 1.0'
                 default_tip_color_rgba:='0 0 1. 1.'
-                motor_id:='6'
-                serial_port:='/dev/pinc-gripper'"
+                "
   >
   <!-- Include links and joints -->
@@ -53,30 +51,4 @@
     <mimic joint="${prefix}gripper" multiplier="0.5" offset="0.0"/>
   </joint>
-  <!-- ros2_control -->
-  <ros2_control name="${prefix}ros2_control" type="system">
-    <hardware>
-      <xacro:if value="${use_mock_hardware}">
-        <plugin>mock_components/GenericSystem</plugin>
-      </xacro:if>
-      <xacro:unless value="${use_mock_hardware}">
-        <plugin>pinc_open_driver/PincOpenDriver</plugin>
-        <param name="port">${serial_port}</param>
-        <param name="baud_rate">1000000</param>
-        <param name="id">${motor_id}</param>
-      </xacro:unless>
-    </hardware>
-    <joint name="${prefix}gripper">
-      <command_interface name="position">
-        <param name="min">-2.44</param>
-        <param name="max">0.0</param>
-      </command_interface>
-      <state_interface name="position">
-        <param name="initial_value">0.0</param>
-      </state_interface>
-      <state_interface name="velocity">
-        <param name="initial_value">0.0</param>
-      </state_interface>
-    </joint>
-  </ros2_control>
   </xacro:macro>
 </robot>
